Commit message: adding filter

File: src/main_bot/description/babydog.ros2_control.xacro (robot description, xacro)
@@ -27,9 +27,7 @@
        hardware_target=gazebo only - it's what leg_pd_controller (the
        low-level layer of the vendored gait stack) actually claims;
-       hardware_target=real exports position/kp/kd instead (matches
-       main_bot_hardware/RealSystem::export_command_interfaces() - RealSystem
-       has NO effort command_interface, declaring one unconditionally here
-       caused controller_manager to reject the hardware with "missing command
-       interfaces: .../effort" on every real bring-up attempt). -->
+       hardware_target=real exports position/velocity/kp/kd/effort instead (matches
+       main_bot_hardware/RealSystem::export_command_interfaces()). "effort" tren real la Tff
+       trong cung khung PD, khong phai effort-only mode. -->
   <ros2_control name="GazeboSimSystem" type="system">
     <hardware>
@@ -46,5 +44,7 @@
       </xacro:if>
       <xacro:if value="${hardware_target == 'real'}">
-        <command_interface name="position"><param name="initial_value">0.0</param></command_interface>
+        <command_interface name="effort"><param name="initial_value">0.0</param></command_interface>
+        <command_interface name="position"><param name="initial_value">0.0</param></command_interface>
+        <command_interface name="velocity"><param name="initial_value">0.0</param></command_interface>
         <command_interface name="kp"><param name="initial_value">0.0</param></command_interface>
         <command_interface name="kd"><param name="initial_value">0.0</param></command_interface>
@@ -59,5 +59,7 @@
       </xacro:if>
       <xacro:if value="${hardware_target == 'real'}">
-        <command_interface name="position"><param name="initial_value">0.0</param></command_interface>
+        <command_interface name="effort"><param name="initial_value">0.0</param></command_interface>
+        <command_interface name="position"><param name="initial_value">0.0</param></command_interface>
+        <command_interface name="velocity"><param name="initial_value">0.0</param></command_interface>
         <command_interface name="kp"><param name="initial_value">0.0</param></command_interface>
         <command_interface name="kd"><param name="initial_value">0.0</param></command_interface>
@@ -72,5 +74,7 @@
       </xacro:if>
       <xacro:if value="${hardware_target == 'real'}">
-        <command_interface name="position"><param name="initial_value">0.0</param></command_interface>
+        <command_interface name="effort"><param name="initial_value">0.0</param></command_interface>
+        <command_interface name="position"><param name="initial_value">0.0</param></command_interface>
+        <command_interface name="velocity"><param name="initial_value">0.0</param></command_interface>
         <command_interface name="kp"><param name="initial_value">0.0</param></command_interface>
         <command_interface name="kd"><param name="initial_value">0.0</param></command_interface>
@@ -85,5 +89,7 @@
       </xacro:if>
       <xacro:if value="${hardware_target == 'real'}">
-        <command_interface name="position"><param name="initial_value">0.0</param></command_interface>
+        <command_interface name="effort"><param name="initial_value">0.0</param></command_interface>
+        <command_interface name="position"><param name="initial_value">0.0</param></command_interface>
+        <command_interface name="velocity"><param name="initial_value">0.0</param></command_interface>
         <command_interface name="kp"><param name="initial_value">0.0</param></command_interface>
         <command_interface name="kd"><param name="initial_value">0.0</param></command_interface>
@@ -98,5 +104,7 @@
       </xacro:if>
       <xacro:if value="${hardware_target == 'real'}">
-        <command_interface name="position"><param name="initial_value">0.0</param></command_interface>
+        <command_interface name="effort"><param name="initial_value">0.0</param></command_interface>
+        <command_interface name="position"><param name="initial_value">0.0</param></command_interface>
+        <command_interface name="velocity"><param name="initial_value">0.0</param></command_interface>
         <command_interface name="kp"><param name="initial_value">0.0</param></command_interface>
         <command_interface name="kd"><param name="initial_value">0.0</param></command_interface>
@@ -111,5 +119,7 @@
       </xacro:if>
       <xacro:if value="${hardware_target == 'real'}">
-        <command_interface name="position"><param name="initial_value">0.0</param></command_interface>
+        <command_interface name="effort"><param name="initial_value">0.0</param></command_interface>
+        <command_interface name="position"><param name="initial_value">0.0</param></command_interface>
+        <command_interface name="velocity"><param name="initial_value">0.0</param></command_interface>
         <command_interface name="kp"><param name="initial_value">0.0</param></command_interface>
         <command_interface name="kd"><param name="initial_value">0.0</param></command_interface>
@@ -124,5 +134,7 @@
       </xacro:if>
       <xacro:if value="${hardware_target == 'real'}">
-        <command_interface name="position"><param name="initial_value">0.0</param></command_interface>
+        <command_interface name="effort"><param name="initial_value">0.0</param></command_interface>
+        <command_interface name="position"><param name="initial_value">0.0</param></command_interface>
+        <command_interface name="velocity"><param name="initial_value">0.0</param></command_interface>
         <command_interface name="kp"><param name="initial_value">0.0</param></command_interface>
         <command_interface name="kd"><param name="initial_value">0.0</param></command_interface>
@@ -137,5 +149,7 @@
       </xacro:if>
       <xacro:if value="${hardware_target == 'real'}">
-        <command_interface name="position"><param name="initial_value">0.0</param></command_interface>
+        <command_interface name="effort"><param name="initial_value">0.0</param></command_interface>
+        <command_interface name="position"><param name="initial_value">0.0</param></command_interface>
+        <command_interface name="velocity"><param name="initial_value">0.0</param></command_interface>
         <command_interface name="kp"><param name="initial_value">0.0</param></command_interface>
         <command_interface name="kd"><param name="initial_value">0.0</param></command_interface>
@@ -150,5 +164,7 @@
       </xacro:if>
       <xacro:if value="${hardware_target == 'real'}">
-        <command_interface name="position"><param name="initial_value">0.0</param></command_interface>
+        <command_interface name="effort"><param name="initial_value">0.0</param></command_interface>
+        <command_interface name="position"><param name="initial_value">0.0</param></command_interface>
+        <command_interface name="velocity"><param name="initial_value">0.0</param></command_interface>
         <command_interface name="kp"><param name="initial_value">0.0</param></command_interface>
         <command_interface name="kd"><param name="initial_value">0.0</param></command_interface>
@@ -163,5 +179,7 @@
       </xacro:if>
       <xacro:if value="${hardware_target == 'real'}">
-        <command_interface name="position"><param name="initial_value">0.0</param></command_interface>
+        <command_interface name="effort"><param name="initial_value">0.0</param></command_interface>
+        <command_interface name="position"><param name="initial_value">0.0</param></command_interface>
+        <command_interface name="velocity"><param name="initial_value">0.0</param></command_interface>
         <command_interface name="kp"><param name="initial_value">0.0</param></command_interface>
         <command_interface name="kd"><param name="initial_value">0.0</param></command_interface>
@@ -176,5 +194,7 @@
       </xacro:if>
       <xacro:if value="${hardware_target == 'real'}">
-        <command_interface name="position"><param name="initial_value">0.0</param></command_interface>
+        <command_interface name="effort"><param name="initial_value">0.0</param></command_interface>
+        <command_interface name="position"><param name="initial_value">0.0</param></command_interface>
+        <command_interface name="velocity"><param name="initial_value">0.0</param></command_interface>
         <command_interface name="kp"><param name="initial_value">0.0</param></command_interface>
         <command_interface name="kd"><param name="initial_value">0.0</param></command_interface>
@@ -189,16 +209,17 @@
       </xacro:if>
       <xacro:if value="${hardware_target == 'real'}">
-        <command_interface name="position"><param name="initial_value">0.0</param></command_interface>
-        <command_interface name="kp"><param name="initial_value">0.0</param></command_interface>
-        <command_interface name="kd"><param name="initial_value">0.0</param></command_interface>
-      </xacro:if>
-      <state_interface name="position"><param name="initial_value">0.0</param></state_interface>
-      <state_interface name="velocity"/>
-      <state_interface name="effort"/>
-    </joint>
-    <!-- No imu_sensor <sensor> block here (yet) - the real robot has no IMU
-         wired to the STM32 yet, so the sim intentionally matches that instead
-         of reading a sensor the real controller can't use. See sensors/imu.xacro
-         and the note at the top of babydog.xacro for how to re-add it later. -->
+        <command_interface name="effort"><param name="initial_value">0.0</param></command_interface>
+        <command_interface name="position"><param name="initial_value">0.0</param></command_interface>
+        <command_interface name="velocity"><param name="initial_value">0.0</param></command_interface>
+        <command_interface name="kp"><param name="initial_value">0.0</param></command_interface>
+        <command_interface name="kd"><param name="initial_value">0.0</param></command_interface>
+      </xacro:if>
+      <state_interface name="position"><param name="initial_value">0.0</param></state_interface>
+      <state_interface name="velocity"/>
+      <state_interface name="effort"/>
+    </joint>
+    <!-- IMU deliberately is not a ros2_control state interface. Both branches
+         publish sensor data through imu_kalman_filter on /imu/data, keeping the
+         real MPU6050 and Gazebo path identical above their raw transports. -->
   </ros2_control>
   <!-- Chi Gazebo doc block nay (moi hardware khac im lang bo qua the <gazebo> khong

File: src/main_bot/description/babydog.xacro (robot description, xacro)
@@ -12,9 +12,6 @@
      knee(pitch), same 3-DOF-per-leg structure as Go1's hip/thigh/calf, just
      renamed - see controllers.yaml's joints/feet_names lists (base_name:
-     "base" is the dummy root link below). No IMU sensor interface yet (real
-     robot doesn't have one wired up yet either) - see sensors/imu.xacro,
-     currently unused; re-add its include in robot.urdf.xacro plus the
-     imu_sensor <ros2_control> block (babydog.ros2_control.xacro) once the
-     real IMU is wired to the STM32. -->
+     "base" is the dummy root link below). imu_link is shared by the Gazebo
+     sensor and the real MPU6050's filtered /imu/data frame. -->
 <robot name="babydog" xmlns:xacro="http://www.ros.org/wiki/xacro">
   <material name="black">

File: src/main_bot/description/robot.urdf.xacro (robot description, xacro)
@@ -1,13 +1,10 @@
 <?xml version="1.0"?>
-<!-- Top-level entry point for the babydog description: this is the file launch
-     files xacro-process, not babydog.xacro directly. Currently just the
-     physical structure - no sensors/*.xacro included yet since the real robot
-     has no IMU/cameras wired up in this phase (stand up / sit down only).
-     Once the real IMU is on the FDCAN link, add back:
-       <xacro:include filename="$(find main_bot)/description/sensors/imu.xacro"/>
-     (and the matching imu_sensor block in babydog.xacro + imu_sensor_broadcaster
-     in config/controllers.yaml - see comments there). -->
+<!-- Top-level entry point for the physical structure, ros2_control and the
+     Gazebo IMU sensor. The real MPU6050 follows a dedicated /imu/raw ->
+     imu_kalman_filter -> /imu/data topic path rather than a ros2_control sensor
+     interface; the same filter consumes /imu/sim_raw in simulation. -->
 <robot name="babydog" xmlns:xacro="http://www.ros.org/wiki/xacro">
   <xacro:include filename="$(find main_bot)/description/babydog.xacro"/>
   <xacro:include filename="$(find main_bot)/description/babydog.ros2_control.xacro"/>
+  <xacro:include filename="$(find main_bot)/description/sensors/imu.xacro"/>
 </robot>

File: src/main_bot/description/sensors/imu.xacro (robot description, xacro)
@@ -1,4 +1,4 @@
 <?xml version="1.0"?>
-<!-- IMU sensor, mounted on imu_link (defined in go1.xacro). -->
+<!-- Gazebo counterpart of the real MPU6050 mounted on imu_link. -->
 <robot xmlns:xacro="http://www.ros.org/wiki/xacro">
   <gazebo reference="imu_link">
@@ -6,20 +6,20 @@
     <sensor name="imu_sensor" type="imu">
       <always_on>true</always_on>
-      <update_rate>1000</update_rate>
-      <visualize>true</visualize>
-      <topic>imu</topic>
-      <!-- Gazebo Classic only (libgazebo_ros_imu_sensor.so). The <sensor> itself is
-           native to gz sim and publishes on gz transport; bridge to ROS with
-           ros_gz_bridge if needed. -->
-      <!-- <plugin filename="libgazebo_ros_imu_sensor.so" name="imu_plugin">
-        <topicName>trunk_imu</topicName>
-        <bodyName>imu_link</bodyName>
-        <updateRateHZ>1000.0</updateRateHZ>
-        <gaussianNoise>0.0</gaussianNoise>
-        <xyzOffset>0 0 0</xyzOffset>
-        <rpyOffset>0 0 0</rpyOffset>
-        <frameName>imu_link</frameName>
-      </plugin> -->
+      <update_rate>100</update_rate>
+      <visualize>false</visualize>
+      <topic>/imu/sim_raw</topic>
       <pose>0 0 0 0 0 0</pose>
+      <imu>
+        <angular_velocity>
+          <x><noise type="gaussian"><mean>0</mean><stddev>0.004</stddev></noise></x>
+          <y><noise type="gaussian"><mean>0</mean><stddev>0.004</stddev></noise></y>
+          <z><noise type="gaussian"><mean>0</mean><stddev>0.004</stddev></noise></z>
+        </angular_velocity>
+        <linear_acceleration>
+          <x><noise type="gaussian"><mean>0</mean><stddev>0.08</stddev></noise></x>
+          <y><noise type="gaussian"><mean>0</mean><stddev>0.08</stddev></noise></y>
+          <z><noise type="gaussian"><mean>0</mean><stddev>0.08</stddev></noise></z>
+        </linear_acceleration>
+      </imu>
     </sensor>
   </gazebo>
